Commit message: relaize path generation

File: assets/temp/temp.urdf (robot description, URDF)
Before this commit: robot model.urdf, 5 links, 4 joints
Links:
- link link_1: geometry collision mesh filename=assets/meshes/stutzmontage/visual/fixture_box.obj scale=0.016094656297717863 0.1 0.02909128158557557; visual mesh filename=assets/meshes/stutzmontage/visual/fixture_box.obj scale=0.016094656297717863 0.1 0.02909128158557557
- link link_2: geometry collision mesh filename=assets/meshes/stutzmontage/visual/fixture_box.obj scale=0.016094656297717863 0.1 0.02909128158557557; visual mesh filename=assets/meshes/stutzmontage/visual/fixture_box.obj scale=0.016094656297717863 0.1 0.02909128158557557
- link link_3: geometry collision mesh filename=assets/meshes/stutzmontage/visual/fixture_box.obj scale=0.005 0.1 0.04598022661269167; visual mesh filename=assets/meshes/stutzmontage/visual/fixture_box.obj scale=0.005 0.1 0.04598022661269167
- link link_4: geometry collision mesh filename=assets/meshes/stutzmontage/visual/fixture_box.obj scale=0.005 0.1 0.04598022661269167; visual mesh filename=assets/meshes/stutzmontage/visual/fixture_box.obj scale=0.005 0.1 0.04598022661269167
Joints:
- joint joint_1: origin xyz=0.0069250018052016225 0 0.018717176746531335 rpy=0.0 0.0 0.0 -> xyz=0.017118944284338168 0 0.014545640792787785 rpy=0.0 0.0 0.0
- joint joint_2: origin xyz=-0.0069250018052016225 0 0.018717176746531335 rpy=0.0 0.0 0.0 -> xyz=-0.017118944284338168 0 0.014545640792787785 rpy=0.0 0.0 0.0
- joint joint_3: origin xyz=0.011925001805201623 0 0.04070532128284822 rpy=0.0 0.0 0.0 -> xyz=0.0276662724331971 0 0.022990113306345834 rpy=0.0 0.0 0.0
- joint joint_4: origin xyz=-0.011925001805201623 0 0.04070532128284822 rpy=0.0 0.0 0.0 -> xyz=-0.0276662724331971 0 0.022990113306345834 rpy=0.0 0.0 0.0

File: assets/temp/temp_nut.urdf (robot description, URDF)
Before this commit: robot model.urdf, 3 links, 2 joints
Links:
- removed link base_nut_link
- added link root
- link link_bot: geometry collision mesh filename=assets/meshes/stutzmontage/visual/Nut_bottom.obj scale=0.01908651606945206 0.01908651606945206 0.017250545655106454; visual mesh filename=assets/meshes/stutzmontage/visual/Nut_bottom.obj scale=0.01908651606945206 0.01908651606945206 0.017250545655106454
- link link_top: geometry collision mesh filename=assets/meshes/stutzmontage/visual/Nut_top.obj scale=0.0417054310965338 0.0417054310965338 0.021383815526490334; visual mesh filename=assets/meshes/stutzmontage/visual/Nut_top.obj scale=0.0417054310965338 0.0417054310965338 0.021383815526490334
Joints:
- joint bot_joint: parent base_nut_link -> root
- joint top_joint: parent base_nut_link -> root

File: assets/temp/temp_screw.urdf (robot description, URDF)
Before this commit: robot model.urdf, 5 links, 4 joints
Links:
- link screw_bot_link: geometry collision mesh filename=assets/meshes/stutzmontage/visual/Screw_bottom.obj scale=0.04425666543665513 0.04425666543665513 0.02803785645024501; visual mesh filename=assets/meshes/stutzmontage/visual/Screw_bottom.obj scale=0.04425666543665513 0.04425666543665513 0.02803785645024501
- link screw_plastic_link: geometry collision mesh filename=assets/meshes/stutzmontage/visual/Screw_plastic.obj scale=0.04425666543665513 0.04425666543665513 0.02803785645024501; visual mesh filename=assets/meshes/stutzmontage/visual/Screw_plastic.obj scale=0.04425666543665513 0.04425666543665513 0.02803785645024501
- link screw_ring_link: geometry collision mesh filename=assets/meshes/stutzmontage/visual/Screw_oring.obj scale=0.04425666543665513 0.04425666543665513 0.02803785645024501; visual mesh filename=assets/meshes/stutzmontage/visual/Screw_oring.obj scale=0.04425666543665513 0.04425666543665513 0.02803785645024501
- link screw_top_link: geometry collision mesh filename=assets/meshes/stutzmontage/visual/Screw_top.obj scale=0.0494868773617393 0.0494868773617393 0.1572344357858577; visual mesh filename=assets/meshes/stutzmontage/visual/Screw_top.obj scale=0.0494868773617393 0.0494868773617393 0.1572344357858577

Commit message: early implenation of RL assembly

File: assets/temp/temp.urdf (robot description, URDF)
Before this commit: robot model.urdf, 5 links, 4 joints
Links:
- link link_1: geometry collision mesh filename=assets/meshes/stutzmontage/visual/fixture_box.obj scale=0.007496473578180205 0.1 0.02819173084119439; visual mesh filename=assets/meshes/stutzmontage/visual/fixture_box.obj scale=0.007496473578180205 0.1 0.02819173084119439
- link link_2: geometry collision mesh filename=assets/meshes/stutzmontage/visual/fixture_box.obj scale=0.007496473578180205 0.1 0.02819173084119439; visual mesh filename=assets/meshes/stutzmontage/visual/fixture_box.obj scale=0.007496473578180205 0.1 0.02819173084119439
- link link_3: geometry collision mesh filename=assets/meshes/stutzmontage/visual/fixture_box.obj scale=0.005 0.1 0.04325896156143998; visual mesh filename=assets/meshes/stutzmontage/visual/fixture_box.obj scale=0.005 0.1 0.04325896156143998
- link link_4: geometry collision mesh filename=assets/meshes/stutzmontage/visual/fixture_box.obj scale=0.005 0.1 0.04325896156143998; visual mesh filename=assets/meshes/stutzmontage/visual/fixture_box.obj scale=0.005 0.1 0.04325896156143998
Joints:
- joint joint_1: origin xyz=0.017118944284338168 0 0.014545640792787785 rpy=0.0 0.0 0.0 -> xyz=0.020508782271023616 0 0.014095865420597195 rpy=0.0 0.0 0.0
- joint joint_2: origin xyz=-0.017118944284338168 0 0.014545640792787785 rpy=0.0 0.0 0.0 -> xyz=-0.020508782271023616 0 0.014095865420597195 rpy=0.0 0.0 0.0
- joint joint_3: origin xyz=0.0276662724331971 0 0.022990113306345834 rpy=0.0 0.0 0.0 -> xyz=0.026757019060113716 0 0.02162948078071999 rpy=0.0 0.0 0.0
- joint joint_4: origin xyz=-0.0276662724331971 0 0.022990113306345834 rpy=0.0 0.0 0.0 -> xyz=-0.026757019060113716 0 0.02162948078071999 rpy=0.0 0.0 0.0

File: assets/temp/temp_nut.urdf (robot description, URDF)
Before this commit: robot model.urdf, 3 links, 2 joints
Links:
- link link_bot: geometry collision mesh filename=assets/meshes/stutzmontage/visual/Nut_bottom.obj scale=0.04325716030211772 0.04325716030211772 0.01657852833430404; visual mesh filename=assets/meshes/stutzmontage/visual/Nut_bottom.obj scale=0.04325716030211772 0.04325716030211772 0.01657852833430404
- link link_top: geometry collision mesh filename=assets/meshes/stutzmontage/visual/Nut_top.obj scale=0.03999468771310285 0.03999468771310285 0.01960414078054761; visual mesh filename=assets/meshes/stutzmontage/visual/Nut_top.obj scale=0.03999468771310285 0.03999468771310285 0.01960414078054761

File: assets/temp/temp_screw.urdf (robot description, URDF)
Before this commit: robot model.urdf, 5 links, 4 joints
Links:
- link screw_bot_link: geometry collision mesh filename=assets/meshes/stutzmontage/visual/Screw_bottom.obj scale=0.042157116738808044 0.042157116738808044 0.025013572568250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; visual mesh filename=assets/meshes/stutzmontage/visual/Screw_bottom.obj scale=0.042157116738808044 0.042157116738808044 0.025013572568250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
- link screw_plastic_link: geometry collision mesh filename=assets/meshes/stutzmontage/visual/Screw_plastic.obj scale=0.042157116738808044 0.042157116738808044 0.025013572568250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; visual mesh filename=assets/meshes/stutzmontage/visual/Screw_plastic.obj scale=0.042157116738808044 0.042157116738808044 0.025013572568250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
- link screw_ring_link: geometry collision mesh filename=assets/meshes/stutzmontage/visual/Screw_oring.obj scale=0.042157116738808044 0.042157116738808044 0.025013572568250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; visual mesh filename=assets/meshes/stutzmontage/visual/Screw_oring.obj scale=0.042157116738808044 0.042157116738808044 0.025013572568250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
- link screw_top_link: geometry collision mesh filename=assets/meshes/stutzmontage/visual/Screw_top.obj scale=0.05991183517108124 0.05991183517108124 0.18049597521616648; visual mesh filename=assets/meshes/stutzmontage/visual/Screw_top.obj scale=0.05991183517108124 0.05991183517108124 0.18049597521616648

File: assets/urdf/rokae_description/xMatePro7.urdf (robot description, URDF)
Before this commit: robot xMatePro7, 12 links, 11 joints
Joints:
- joint finger_joint1: limit lower=0.0 upper=0.04 effort=20 velocity=0.2 -> lower=0.0 upper=0.04 effort=200 velocity=0.2
- joint finger_joint2: limit lower=0.0 upper=0.04 effort=20 velocity=0.2 -> lower=0.0 upper=0.04 effort=300 velocity=0.01

Commit message: assembly_ur5e

File: assets/temp/temp.urdf (robot description, URDF)
Before this commit: robot model.urdf, 5 links, 4 joints
Links:
- link link_1: geometry collision mesh filename=assets/meshes/stutzmontage/visual/fixture_box.obj scale=0.005092111718412978 0.1 0.05142787987854228; visual mesh filename=assets/meshes/stutzmontage/visual/fixture_box.obj scale=0.005092111718412978 0.1 0.05142787987854228
- link link_2: geometry collision mesh filename=assets/meshes/stutzmontage/visual/fixture_box.obj scale=0.005092111718412978 0.1 0.05142787987854228; visual mesh filename=assets/meshes/stutzmontage/visual/fixture_box.obj scale=0.005092111718412978 0.1 0.05142787987854228
- link link_3: geometry collision mesh filename=assets/meshes/stutzmontage/visual/fixture_box.obj scale=0.005 0.1 0.08905381179501778; visual mesh filename=assets/meshes/stutzmontage/visual/fixture_box.obj scale=0.005 0.1 0.08905381179501778
- link link_4: geometry collision mesh filename=assets/meshes/stutzmontage/visual/fixture_box.obj scale=0.005 0.1 0.08905381179501778; visual mesh filename=assets/meshes/stutzmontage/visual/fixture_box.obj scale=0.005 0.1 0.08905381179501778
Joints:
- joint joint_1: origin xyz=0.020508782271023616 0 0.014095865420597195 rpy=0.0 0.0 0.0 -> xyz=0.013693161164097706 0 0.02571393993927114 rpy=0.0 0.0 0.0
- joint joint_2: origin xyz=-0.020508782271023616 0 0.014095865420597195 rpy=0.0 0.0 0.0 -> xyz=-0.013693161164097706 0 0.02571393993927114 rpy=0.0 0.0 0.0
- joint joint_3: origin xyz=0.026757019060113716 0 0.02162948078071999 rpy=0.0 0.0 0.0 -> xyz=0.018739217023304194 0 0.04452690589750889 rpy=0.0 0.0 0.0
- joint joint_4: origin xyz=-0.026757019060113716 0 0.02162948078071999 rpy=0.0 0.0 0.0 -> xyz=-0.018739217023304194 0 0.04452690589750889 rpy=0.0 0.0 0.0

File: assets/temp/temp_nut.urdf (robot description, URDF)
Before this commit: robot model.urdf, 3 links, 2 joints
Links:
- link link_bot: geometry collision mesh filename=assets/meshes/stutzmontage/visual/Nut_bottom.obj scale=0.02561094984458378 0.02561094984458378 0.033937298497499234; visual mesh filename=assets/meshes/stutzmontage/visual/Nut_bottom.obj scale=0.02561094984458378 0.02561094984458378 0.033937298497499234
- link link_top: geometry collision mesh filename=assets/meshes/stutzmontage/visual/Nut_top.obj scale=0.024909341658661228 0.024909341658661228 0.041642256564556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; visual mesh filename=assets/meshes/stutzmontage/visual/Nut_top.obj scale=0.024909341658661228 0.024909341658661228 0.041642256564556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

File: assets/temp/temp_screw.urdf (robot description, URDF)
Before this commit: robot model.urdf, 5 links, 4 joints
Links:
- link screw_bot_link: geometry collision mesh filename=assets/meshes/stutzmontage/visual/Screw_bottom.obj scale=0.023643282944720602 0.023643282944720602 0.062463965403822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; visual mesh filename=assets/meshes/stutzmontage/visual/Screw_bottom.obj scale=0.023643282944720602 0.023643282944720602 0.062463965403822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
- link screw_plastic_link: geometry collision mesh filename=assets/meshes/stutzmontage/visual/Screw_plastic.obj scale=0.023643282944720602 0.023643282944720602 0.062463965403822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; visual mesh filename=assets/meshes/stutzmontage/visual/Screw_plastic.obj scale=0.023643282944720602 0.023643282944720602 0.062463965403822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
- link screw_ring_link: geometry collision mesh filename=assets/meshes/stutzmontage/visual/Screw_oring.obj scale=0.023643282944720602 0.023643282944720602 0.062463965403822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; visual mesh filename=assets/meshes/stutzmontage/visual/Screw_oring.obj scale=0.023643282944720602 0.023643282944720602 0.062463965403822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
- link screw_top_link: geometry collision mesh filename=assets/meshes/stutzmontage/visual/Screw_top.obj scale=0.07106022933319493 0.07106022933319493 0.05443311985069603; visual mesh filename=assets/meshes/stutzmontage/visual/Screw_top.obj scale=0.07106022933319493 0.07106022933319493 0.05443311985069603
